File: Disp_Sec_V_1/Disp_Sec_V_1.kicad_pcb (KiCad board)
At the start: 2 copper layers, 42 parts, among them J1 Conn_01x02, J2 Conn_01x02, J3 Conn_01x02, K1 FINDER-36.11, K2 FINDER-36.11, K3 FINDER-36.11, Q1 Q_NPN_BCE, Q2 Q_NPN_BCE, Q3 Q_NPN_BCE, Q4 Q_NPN_BCE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

Commit message: Avances PCB
Parts:
- added G***: LOGO, Disp_Sec_V_1:isolse, F.Cu at (134.0, 81.0)
- added G***: LOGO, Disp_Sec_V_1:Spidey, F.Cu at (192.0, 80.0)
- J1: value Conn_01x02 -> DC Supply
- J2: value Conn_01x02 -> Contacto A (N.O)
- J3: value Conn_01x02 -> Contacto F (N.0)
- moved R6 134.8 mm to (78.0, 121.0), turned to 90 degrees
- moved J2 131.5 mm to (82.0, 97.0), turned to 270 degrees
- moved F1 123.6 mm to (221.0, 68.9), turned to 180 degrees
- moved Q4 105.3 mm to (90.0, 111.0), turned to 270 degrees
- moved R10 95.9 mm to (95.0, 120.0), turned to 180 degrees
- moved K2 92.7 mm to (87.0, 83.0), turned to 90 degrees
- moved D3 91.1 mm to (86.0, 92.0)
- moved R2 90.6 mm to (112.0, 110.0)
- moved J3 87.5 mm to (117.0, 119.0)
- moved D11 86.0 mm to (128.0, 121.0)
- moved D4 85.3 mm to (92.0, 96.0), turned to 270 degrees
- moved U4 79.6 mm to (213.6, 114.5)
- moved D8 78.1 mm to (132.0, 106.0), turned to 270 degrees
- moved D6 77.1 mm to (124.0, 106.0), turned to 180 degrees
- moved D10 75.6 mm to (101.0, 98.0), turned to 90 degrees
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Connections:
- U1 pad 14: Net-(U1-Pad14) -> GND
- U1 pad 24: Net-(U1-Pad24) -> GND
Routing:
- net GND: track 0.00 -> 451.4 mm
- net +12V: track 0.00 -> 291.0 mm
- net +3V3: track 0.00 -> 137.0 mm
- net /RST: track 0.00 -> 117.9 mm
- net /ALARMA: track 0.00 -> 88.5 mm
- net Net-(D8-Pad2): track 0.00 -> 81.3 mm
- net /FALLA: track 0.00 -> 65.7 mm
- net /CE: track 0.00 -> 56.6 mm
- net /VCC_CONT: track 0.00 -> 51.9 mm
- net /CSN: track 0.00 -> 50.9 mm
- net /MISO: track 0.00 -> 45.6 mm
- net /SCK: track 0.00 -> 43.9 mm
- net /MOSI: track 0.00 -> 43.9 mm
- net Net-(D7-Pad2): track 0.00 -> 38.4 mm
- net Net-(D2-Pad2): track 0.00 -> 35.7 mm
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Other:
- board outline added: 153 x 68 mm
- net class Default: clearance 0.2 -> 0.4
- rule trace_clearance: 0.2 -> 0.4
- board text added: "+24 VDC"
- board text added: "C. ALARMA"
- board text added: "C. FALLA"
