File: Disp_Sec_V_1/Disp_Sec_V_1.kicad_pcb (KiCad board)
At the start: 2 copper layers, 146 x 62 mm, 49 parts, among them J1 DC Supply, J2 Contacto A (N.O), J3 Contacto F (N.0), K1 FINDER-36.11, K2 FINDER-36.11, K3 FINDER-36.11, Q1 Q_NPN_BCE, Q2 Q_NPN_BCE, Q3 Q_NPN_BCE, Q4 Q_NPN_BCE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

Commit message: Correcciones Finales
Parts:
- removed G***: LOGO, Disp_Sec_V_1:isolse
- removed G***: LOGO, Disp_Sec_V_1:C.FALLA
- removed G***: LOGO, Disp_Sec_V_1:C.ALARMA
- removed G***: LOGO, Disp_Sec_V_1:DC
- removed REF** (x3): Fiducial_0.5mm_Mask1.5mm, Fiducial:Fiducial_0.5mm_Mask1.5mm
- added FID1: Fiducial, Fiducial:Fiducial_1mm_Mask2mm, F.Cu at (146.0, 121.0)
- added FID2: Fiducial, Fiducial:Fiducial_1mm_Mask2mm, F.Cu at (132.0, 65.0)
- added FID3: Fiducial, Fiducial:Fiducial_1mm_Mask2mm, F.Cu at (222.0, 76.0)
- added H1: MountingHole, MountingHole:MountingHole_2.5mm, F.Cu at (185.0, 118.5)
- added H2: MountingHole, MountingHole:MountingHole_2.5mm, F.Cu at (121.0, 66.0)
- added H3: MountingHole, MountingHole:MountingHole_2.5mm, F.Cu at (185.0, 66.0)
- added H4: MountingHole, MountingHole:MountingHole_2.5mm, F.Cu at (108.0, 115.5)
- added TP1: TestPoint, TestPoint:TestPoint_Loop_D1.80mm_Drill1.0mm_Beaded, F.Cu at (184.5, 80.0)
- added TP2: TestPoint, TestPoint:TestPoint_Loop_D1.80mm_Drill1.0mm_Beaded, F.Cu at (160.5, 119.0)
- added TP3: TestPoint, TestPoint:TestPoint_Loop_D1.80mm_Drill1.0mm_Beaded, F.Cu at (156.2, 119.0)
- added TP4: TestPoint, TestPoint:TestPoint_Loop_D1.80mm_Drill1.0mm_Beaded, F.Cu at (152.0, 119.0)
- added U5: DEEPCONTROL_LOGO, Disp_Sec_V_1:DC, F.Cu at (140.0, 86.0)
- added U6: isolseLOGO, Disp_Sec_V_1:isolse, F.Cu at (196.0, 87.0)
- added U7: Contacto_Falla, Disp_Sec_V_1:C.FALLA, F.Cu at (130.0, 121.0)
- added U8: Contacto_Alarma, Disp_Sec_V_1:C.ALARMA, F.Cu at (84.0, 114.0)
- D1, D7, D8: value D -> 1N5349B
- D2: value D -> 1N5359B
- D3, D5: value Diode -> SR2100
- D4, D6: value diode -> SR2100
- Q1, Q2, Q3, Q4, Q5, Q6: value Q_NPN_BCE -> BC337
- moved Q2 5.10 mm to (194.0, 118.0)
- moved Q6 3.16 mm to (180.0, 96.0), turned to 0 degrees
- moved J1 1.82 mm to (191.0, 69.0)
- moved Q3 1.58 mm to (180.5, 86.5), turned to 0 degrees
- moved D6 1.00 mm to (124.0, 100.0)
Routing:
- net GND: track 479.5 -> 1.36 mm
- net +12V: track 392.6 -> 1.00 mm
- net Net-(D1-Pad2): track 30.3 -> 53.8 mm
- net /FALLA: track 60.7 -> 70.2 mm
- net Net-(D9-Pad2): track 32.0 -> 22.9 mm
- net /VCC_CONT: track 66.2 -> 72.9 mm
- net Net-(Q2-Pad1): track 8.26 -> 13.4 mm
- net /RST: track 100.9 -> 96.5 mm
- net +3V3: track 113.6 -> 117.3 mm
- net Net-(D2-Pad2): track 28.9 -> 25.4 mm
- net Net-(Q1-Pad2): track 15.5 -> 18.1 mm
- net /MISO: track 45.6 -> 48.2 mm
- net Net-(Q6-Pad1): track 6.54 -> 9.13 mm
- net /CE: track 56.0 -> 58.2 mm
- net Net-(D11-Pad1): track 28.6 -> 30.6 mm
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- added copper zone on F.Cu, net +12V
- added copper zone on B.Cu, net GND
Other:
- net class Default: clearance 0.4 -> 0.6
- rule trace_clearance: 0.4 -> 0.6
- board text added: "+12V"
- board text added: "+3.3V"
- board text added: "+Vin"
- board text added: "El diseno se realiza con los siguientes parametros: * Ancho de pista de 0.8 mm. * Pads de COBRE con recubrimiento de FLUX. * Mascara antisoldante verde Estano-Plomo. * Grilla de 1mm para Posicionamiento y 0,5mm para Routeo. * Pad minimo 0,7 mm * Espesor de placa (standard) 1.6 mm. * Espesor de cobre (standard) 35 um. * Material de Sustrato: FR4. * DOBLE FAZ con componentes unicamente en la capa f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"
- board text added: "GND"
- board text added: "In"
- board text added: "Out"
- board text added: "VCC_CONT"
- board text removed: "El diseno se realiza con los siguientes parametros: * Ancho de pista de 0.8 mm. * Pads de COBRE con recubrimiento de FLUX. * Mascara antisoldante verde Estano-Plomo. * Espesor de placa (standard) 1.6 mm. * Espesor de cobre (standard) 35 um. * Material de Sustrato: FR4. * DOBLE FAZ con componentes unicamente en la capa frontal. * Se desea mantener un margen de 2 mm en toda la periferia de la placa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"

Commit message: Correcciones de Segunda Revision
Parts:
- F1: value Fuse -> 100mA (5 x 20); footprint Fuse_Holders_and_Fuses:Fuseholder5x20_horiz_open_inline_Type-I -> Disp_Sec_V_1:Fuse
- moved F1 9.72 mm to (211.2, 68.9)
Routing:
- net Net-(D8-Pad2): track 34.2 -> 40.4 mm
Other:
- board text added: "El diseno se realiza con los siguientes parametros: * Ancho de pista de 0.8 mm. * Pads de COBRE con recubrimiento de FLUX. * Mascara antisoldante verde. * Terminacion superficial de pads HASL. * Grilla de 1mm para Posicionamiento y 0,5mm para Routeo. * Pad minimo 0,7 mm * Espesor de placa (standard) 1.6 mm. * Espesor de cobre (standard) 35 um. * Material de Sustrato: FR4. * DOBLE FAZ con componen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"
- board text removed: "El diseno se realiza con los siguientes parametros: * Ancho de pista de 0.8 mm. * Pads de COBRE con recubrimiento de FLUX. * Mascara antisoldante verde Estano-Plomo. * Grilla de 1mm para Posicionamiento y 0,5mm para Routeo. * Pad minimo 0,7 mm * Espesor de placa (standard) 1.6 mm. * Espesor de cobre (standard) 35 um. * Material de Sustrato: FR4. * DOBLE FAZ con componentes unicamente en la capa f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"
